File: MultiVib.sch (KiCad schematic (older format))
At the start: 11 parts

Commit message: Add files via upload
Parts:
- removed Q? (x2): BC548, Package_TO_SOT_THT:TO-92_Inline, symbol Transistor_BJT:BC548
- added U?: BCM586DS, symbol New_Library:BCM586DS
Connections:
- net at C?.1, R?.2: now also U?.4 (C_TR1)
- net at C?.2, R?.2: now also U?.5 (B_TR2)
- net at C?.2, R?.2: now also U?.2 (B_TR1)
- net at C?.1, R?.2: now also U?.3 (C_TR2)
- net at BT?.2 (-): now also U?.1 (E_TR1), U?.6 (E_TR2)
Changed lines of the file:
@@
 encoding utf-8
 Sheet 1 1
-Title "MultiVib"
+Title "MultiVib with BCM586DS"
 Date ""
 Rev ""
@@
 $EndComp
 $Comp
-L Transistor_BJT:BC548 Q?
-U 1 1 5E67AB5D
-P 3650 3150
-F 0 "Q?" H 3841 3196 50  0000 L CNN
-F 1 "BC548" H 3841 3105 50  0000 L CNN
-F 2 "Package_TO_SOT_THT:TO-92_Inline" H 3850 3075 50  0001 L CIN
-F 3 "http://www.fairchildsemi.com/ds/BC/BC547.pdf" H 3650 3150 50  0001 L CNN
-	1    3650 3150
-	-1   0    0    -1
-$EndComp
-$Comp
-L Transistor_BJT:BC548 Q?
-U 1 1 5E67ABA5
-P 5250 3150
-F 0 "Q?" H 5441 3196 50  0000 L CNN
-F 1 "BC548" H 5441 3105 50  0000 L CNN
-F 2 "Package_TO_SOT_THT:TO-92_Inline" H 5450 3075 50  0001 L CIN
-F 3 "http://www.fairchildsemi.com/ds/BC/BC547.pdf" H 5250 3150 50  0001 L CNN
-	1    5250 3150
-	1    0    0    -1
-$EndComp
-$Comp
 L Device:CP1 C?
 U 1 1 5E67AD68
@@
 	5350 2650 5250 2650
 Wire Wire Line
-	5350 2650 5350 2950
-Connection ~ 5350 2650
-Wire Wire Line
-	5350 3350 5350 3650
-Wire Wire Line
-	5350 3650 3550 3650
-Wire Wire Line
-	3550 3650 3550 3350
-Wire Wire Line
-	3550 2950 3550 2650
-Connection ~ 3550 2650
-Wire Wire Line
-	4950 2650 4550 2650
-Wire Wire Line
-	4550 2650 4550 3150
-Wire Wire Line
-	4550 3150 3850 3150
-Wire Wire Line
-	4000 2650 4000 2900
-Wire Wire Line
-	4000 2900 4750 2900
-Wire Wire Line
-	4750 2900 4750 3150
-Wire Wire Line
-	4750 3150 5050 3150
+	4950 2650 4800 2650
 Wire Wire Line
 	4000 2650 4000 2250
-Connection ~ 4000 2650
-Wire Wire Line
-	4550 2650 4550 2400
-Wire Wire Line
-	4550 2400 4800 2400
-Wire Wire Line
-	4800 2400 4800 2250
-Connection ~ 4550 2650
 Wire Wire Line
 	4800 1950 4800 1100
@@
 	4800 1100 5350 1100
 Wire Wire Line
-	3550 3650 2600 3650
-Wire Wire Line
-	2600 3650 2600 2450
-Connection ~ 3550 3650
-Wire Wire Line
 	2600 2050 2600 1100
 Wire Wire Line
 	2600 1100 3550 1100
 Connection ~ 3550 1100
+$Comp
+L New_Library:BCM586DS U?
+U 1 1 5E67D9BA
+P 4550 3150
+F 0 "U?" H 4550 2785 50  0000 C CNN
+F 1 "BCM586DS" H 4550 2876 50  0000 C CNN
+F 2 "" H 4550 3400 50  0001 C CNN
+F 3 "" H 4550 3400 50  0001 C CNN
+	1    4550 3150
+	-1   0    0    1
+$EndComp
+Wire Wire Line
+	5100 3300 5100 3600
+Wire Wire Line
+	4050 2650 4000 2650
+Connection ~ 4000 2650
+Wire Wire Line
+	3550 3300 3550 2650
+Connection ~ 3550 2650
+Wire Wire Line
+	2600 3600 3250 3600
+Wire Wire Line
+	4050 2650 4050 3150
+Wire Wire Line
+	4950 3000 5350 3000
+Wire Wire Line
+	5350 3000 5350 2650
+Connection ~ 5350 2650
+Wire Wire Line
+	4950 3150 5150 3150
+Wire Wire Line
+	5150 3150 5150 2800
+Wire Wire Line
+	5150 2800 4800 2800
+Wire Wire Line
+	4800 2800 4800 2650
+Wire Wire Line
+	4800 2250 4800 2650
+Connection ~ 4800 2650
+Wire Wire Line
+	4950 3300 5100 3300
+Wire Wire Line
+	3550 3300 4150 3300
+Wire Wire Line
+	4050 3150 4150 3150
+Wire Wire Line
+	4150 3000 3250 3000
+Wire Wire Line
+	3250 3000 3250 3600
+Connection ~ 3250 3600
+Wire Wire Line
+	3250 3600 5100 3600
+Wire Wire Line
+	2600 2450 2600 3600
 $EndSCHEMATC
